File: CANBus/Hardware/CAN_Shield/CAN_Shield.kicad_pcb (KiCad board)
At the start: 2 copper layers, 101.6 x 53.3 mm, 13 parts, among them J1 Power, J2 PWM, J3 Analog, J4 PWM, J5 Analog, J6 Communication, J7 Digital

Commit message: feat: added PCB design
Parts:
- added C1: 0.1u, Capacitor_SMD:C_0805_2012Metric_Pad1.18x1.45mm_HandSolder, F.Cu at (132.4, 77.7)
- added C2: 0.1u, Capacitor_SMD:C_0805_2012Metric_Pad1.18x1.45mm_HandSolder, F.Cu at (124.3, 85.8)
- added J8: Screw_Terminal_01x02, TerminalBlock:TerminalBlock_bornier-2_P5.08mm, F.Cu at (104.2, 79.7)
- added JP2: SolderJumper_2_Bridged, Connector_PinHeader_2.54mm:PinHeader_1x02_P2.54mm_Vertical, F.Cu at (115.1, 74.6)
- added R1: 60, Resistor_SMD:R_0201_0603Metric, F.Cu at (111.5, 79.1)
- added R2: 60, Resistor_SMD:R_0201_0603Metric, F.Cu at (111.5, 75.2)
- added U2: TCAN1051HGV, Package_SO:SOIC-8_3.9x4.9mm_P1.27mm, F.Cu at (126.3, 77.3)
Connections:
- J5 pad 7: /A14 -> /CANRX0_DUE/GIGA
- J5 pad 8: /A15 -> /CANTX0_DUE/GIGA
Routing:
- net /CANRX0_DUE/GIGA: track 0.00 -> 81.0 mm
- net /CANTX0_DUE/GIGA: track 0.00 -> 80.2 mm, vias 0 -> 1
- net /*2: track 0.00 -> 63.5 mm
- net +3V3: track 0.00 -> 32.6 mm, vias 0 -> 2
- net +5V: track 0.00 -> 29.8 mm
- net Net-(J8-Pin_2): track 0.00 -> 22.3 mm
- net Net-(J8-Pin_1): track 0.00 -> 21.8 mm
- net Net-(JP2-B): track 0.00 -> 10.7 mm, vias 0 -> 1
- net Net-(JP2-A): track 0.00 -> 3.73 mm
- net GND: vias 0 -> 27
- added copper zone on B.Cu, net GND
- added copper zone on F.Cu, net GND
