File: CANBus/Hardware/CAN_Shield_UNO/CAN_Shield_UNO.kicad_pcb (KiCad board)
At the start: 2 copper layers, 68.6 x 53.3 mm, 8 parts, among them J1 Power, J2 Digital/PWM, J3 Analog, J4 Digital/PWM

Commit message: feat: added PCB design
Parts:
- added C1: 0.1u, Capacitor_SMD:C_0805_2012Metric_Pad1.18x1.45mm_HandSolder, F.Cu at (137.3, 87.5)
- added J5: ~, Connector_PinHeader_2.54mm:PinHeader_2x04_P2.54mm_Vertical, F.Cu at (128.9, 79.4)
- added J7: Screw_Terminal_01x02, TerminalBlock:TerminalBlock_bornier-2_P5.08mm, F.Cu at (164.6, 80.4)
- added JP1: SolderJumper_2_Bridged, Connector_PinHeader_2.54mm:PinHeader_1x02_P2.54mm_Vertical, F.Cu at (156.9, 80.2)
- added R2: 60, Resistor_SMD:R_0201_0603Metric, F.Cu at (149.7, 82.2)
- added R3: 60, Resistor_SMD:R_0201_0603Metric, F.Cu at (149.6, 84.2)
- added U2: TCAN1051HGV, Package_SO:SOIC-8_3.9x4.9mm_P1.27mm, F.Cu at (142.2, 83.2)
Connections:
- J2 pad 5: /13 -> /CRX0_WIFI
- J2 pad 8: /*10 -> /CTX0_WIFI
- J4 pad 3: /*5 -> /CRX0_MINIMA
- J4 pad 4: /4 -> /CTX0_MINIMA
Routing:
- net /CTX0_MINIMA: track 0.00 -> 70.7 mm
- net /CRX0_MINIMA: track 0.00 -> 58.1 mm, vias 0 -> 1
- net /CTX0_WIFI: track 0.00 -> 49.3 mm, vias 0 -> 1
- net /2: track 0.00 -> 45.3 mm
- net /CRX0_WIFI: track 0.00 -> 30.2 mm, vias 0 -> 1
- net +5V: track 0.00 -> 22.8 mm
- net Net-(J7-Pin_1): track 0.00 -> 20.8 mm
- net Net-(J7-Pin_2): track 0.00 -> 20.6 mm
- net Net-(JP1-A): track 0.00 -> 14.5 mm, vias 0 -> 1
- net Net-(J5-Pin_7): track 0.00 -> 11.1 mm
- net Net-(J5-Pin_5): track 0.00 -> 11.0 mm
- net Net-(JP1-B): track 0.00 -> 6.04 mm
- net GND: vias 0 -> 37
- added copper zone on B.Cu, net GND
- added copper zone on F.Cu, net GND
