File: CANBus/Hardware/CAN_Shield_UNO/CAN_Shield_UNO.kicad_pcb (KiCad board)
At the start: 2 copper layers, 68.6 x 53.3 mm, 39 parts, among them J1 Power, J2 Digital/PWM, J3 Analog, J4 Digital/PWM, J7 Screw_Terminal_01x02, U2 TCAN1051HGV

Commit message: fix: change routing
Parts:
- moved kibuzzard-66182706 5.24 mm to (125.1, 84.2)
- moved kibuzzard-66182736 5.22 mm to (124.3, 86.7)
- moved kibuzzard-6618272A 5.12 mm to (124.2, 81.6)
- moved kibuzzard-6618271B 5.06 mm to (125.0, 79.1)
- moved kibuzzard-661826AE 2.88 mm to (139.6, 84.2)
- moved kibuzzard-661826C2 2.68 mm to (139.4, 81.5)
Connections:
- C2 pad 1: +3V3 -> +5V
- J5 pad 1: /CRX0_WIFI -> /CTX0_WIFI
- J5 pad 2: /CRX0_MINIMA -> /CTX0_MINIMA
- J5 pad 3: /CTX0_WIFI -> /CRX0_WIFI
- J5 pad 4: /CTX0_MINIMA -> /CRX0_MINIMA
- U2 pad 5: +3V3 -> +5V
Routing:
- net /CTX0_MINIMA: track 61.2 -> 42.3 mm
- net /CTX0_WIFI: track 47.0 -> 31.6 mm
- net /CRX0_MINIMA: track 57.1 -> 48.2 mm
- net /CRX0_WIFI: track 32.7 -> 36.3 mm
- net Net-(J5-Pin_5): track 12.2 -> 8.88 mm
- net Net-(J5-Pin_7): track 12.3 -> 8.97 mm
Changed lines of the file:
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@@
 			(at 1.27 9.95 0)
 			(layer "F.Fab")
+			(hide yes)
 			(effects
 				(font
@@
 			(layers "*.Cu" "*.Mask")
 			(remove_unused_layers no)
-			(net 11 "/CRX0_WIFI")
+			(net 17 "/CTX0_WIFI")
 			(pinfunction "Pin_1")
 			(pintype "passive")
@@
 			(layers "*.Cu" "*.Mask")
 			(remove_unused_layers no)
-			(net 22 "/CRX0_MINIMA")
+			(net 19 "/CTX0_MINIMA")
 			(pinfunction "Pin_2")
 			(pintype "passive")
@@
 			(layers "*.Cu" "*.Mask")
 			(remove_unused_layers no)
-			(net 17 "/CTX0_WIFI")
+			(net 11 "/CRX0_WIFI")
 			(pinfunction "Pin_3")
 			(pintype "passive")
@@
 			(layers "*.Cu" "*.Mask")
 			(remove_unused_layers no)
-			(net 19 "/CTX0_MINIMA")
+			(net 22 "/CRX0_MINIMA")
 			(pinfunction "Pin_4")
 			(pintype "passive")
@@
 			)
 		)
-		(property "LCSC#" "C424093"
+		(property "LCSC#" ""
 			(at 0 0 0)
 			(unlocked yes)
@@
 			)
 		)
-		(property "Proveedor" "LCSC"
+		(property "Proveedor" "MOUSER"
 			(at 0 0 0)
 			(unlocked yes)
@@
 			)
 		)
-		(property "manf#" "MCP73831T-2ACI/OT"
+		(property "manf#" "595-TCAN1051HGVDR"
 			(at 0 0 0)
 			(unlocked yes)
@@
 			(layers "F.Cu" "F.Paste" "F.Mask")
 			(roundrect_rratio 0.25)
-			(net 26 "+3V3")
+			(net 3 "+5V")
 			(pinfunction "VIO")
 			(pintype "input")
@@
 	(footprint "kibuzzard-6618271B"
 		(layer "F.Cu")
-		(at 125.48 84.11)
+		(at 124.95 79.075)
 		(descr "Generated with KiBuzzard")
 		(tags "kb_params=eyJBbGlnbm1lbnRDaG9pY2UiOiAiQ2VudGVyIiwgIkNhcExlZnRDaG9pY2UiOiAiKCIsICJDYXBSaWdodENob2ljZSI6ICI+IiwgIkZvbnRDb21ib0JveCI6ICJtcGx1cy0xbW4tbWVkaXVtIiwgIkhlaWdodEN0cmwiOiAiMSIsICJMYXllckNvbWJvQm94IjogIkYuU2lsa1MiLCAiTXVsdGlMaW5lVGV4dCI6ICJDQU5UWF9XSUZJIiwgIlBhZGRpbmdCb3R0b21DdHJsIjogIiIsICJQYWRkaW5nTGVmdEN0cmwiOiAiIiwgIlBhZGRpbmdSaWdodEN0cmwiOiAiIiwgIlBhZGRpbmdUb3BDdHJsIjogIiIsICJXaWR0aEN0cmwiOiAiIn0=")
@@
 	(footprint "kibuzzard-66182736"
 		(layer "F.Cu")
-		(at 124.56 81.51)
+		(at 124.325 86.725)
 		(descr "Generated with KiBuzzard")
 		(tags "kb_params=eyJBbGlnbm1lbnRDaG9pY2UiOiAiQ2VudGVyIiwgIkNhcExlZnRDaG9pY2UiOiAiKCIsICJDYXBSaWdodENob2ljZSI6ICI+IiwgIkZvbnRDb21ib0JveCI6ICJtcGx1cy0xbW4tbWVkaXVtIiwgIkhlaWdodEN0cmwiOiAiMSIsICJMYXllckNvbWJvQm94IjogIkYuU2lsa1MiLCAiTXVsdGlMaW5lVGV4dCI6ICJDQU5SWF9NSU5JTUEiLCAiUGFkZGluZ0JvdHRvbUN0cmwiOiAiIiwgIlBhZGRpbmdMZWZ0Q3RybCI6ICIiLCAiUGFkZGluZ1JpZ2h0Q3RybCI6ICIiLCAiUGFkZGluZ1RvcEN0cmwiOiAiIiwgIldpZHRoQ3RybCI6ICIifQ==")
@@
 	(footprint "kibuzzard-661826C2"
 		(layer "F.Cu")
-		(at 139.7 84.12)
+		(at 139.425 81.45)
 		(descr "Generated with KiBuzzard")
 		(tags "kb_params=eyJBbGlnbm1lbnRDaG9pY2UiOiAiQ2VudGVyIiwgIkNhcExlZnRDaG9pY2UiOiAiPCIsICJDYXBSaWdodENob2ljZSI6ICIpIiwgIkZvbnRDb21ib0JveCI6ICJtcGx1cy0xbW4tbWVkaXVtIiwgIkhlaWdodEN0cmwiOiAiMSIsICJMYXllckNvbWJvQm94IjogIkYuU2lsa1MiLCAiTXVsdGlMaW5lVGV4dCI6ICJDQU5UWCIsICJQYWRkaW5nQm90dG9tQ3RybCI6ICIiLCAiUGFkZGluZ0xlZnRDdHJsIjogIiIsICJQYWRkaW5nUmlnaHRDdHJsIjogIiIsICJQYWRkaW5nVG9wQ3RybCI6ICIiLCAiV2lkdGhDdHJsIjogIiJ9")
@@
 	(footprint "kibuzzard-661826AE"
 		(layer "F.Cu")
-		(at 139.7 81.37)
+		(at 139.55 84.25)
 		(descr "Generated with KiBuzzard")
 		(tags "kb_params=eyJBbGlnbm1lbnRDaG9pY2UiOiAiQ2VudGVyIiwgIkNhcExlZnRDaG9pY2UiOiAiPCIsICJDYXBSaWdodENob2ljZSI6ICIpIiwgIkZvbnRDb21ib0JveCI6ICJtcGx1cy0xbW4tbWVkaXVtIiwgIkhlaWdodEN0cmwiOiAiMSIsICJMYXllckNvbWJvQm94IjogIkYuU2lsa1MiLCAiTXVsdGlMaW5lVGV4dCI6ICJDQU5SWCIsICJQYWRkaW5nQm90dG9tQ3RybCI6ICIiLCAiUGFkZGluZ0xlZnRDdHJsIjogIiIsICJQYWRkaW5nUmlnaHRDdHJsIjogIiIsICJQYWRkaW5nVG9wQ3RybCI6ICIiLCAiV2lkdGhDdHJsIjogIiJ9")
@@
 			)
 		)
-		(property "LCSC#" "C492401"
+		(property "LCSC#" ""
 			(at 0 0 0)
 			(unlocked yes)
@@
 			)
 		)
-		(property "Proveedor" "LCSC"
+		(property "Proveedor" ""
 			(at 0 0 0)
 			(unlocked yes)
@@
 			)
 		)
-		(property "manf#" "PZ254V-11-02P "
+		(property "manf#" ""
 			(at 0 0 0)
 			(unlocked yes)
@@
 		(sheetfile "CAN_Shield_UNO.kicad_sch")
 		(zone_connect 1)
-		(attr exclude_from_pos_files exclude_from_bom)
+		(attr exclude_from_pos_files exclude_from_bom dnp)
 		(net_tie_pad_groups "1, 2")
 		(fp_poly
@@
 			)
 		)
-		(property "manf#" " 0805B104K500NT"
+		(property "manf#" "0805B104K500NT"
 			(at 0 0 0)
 			(unlocked yes)
@@
 			(layers "F.Cu" "F.Paste" "F.Mask")
 			(roundrect_rratio 0.212766)
-			(net 26 "+3V3")
+			(net 3 "+5V")
 			(pintype "passive")
 		)
@@
 	(footprint "kibuzzard-66182706"
 		(layer "F.Cu")
-		(at 125.55 78.93)
+		(at 125.075 84.15)
 		(descr "Generated with KiBuzzard")
 		(tags "kb_params=eyJBbGlnbm1lbnRDaG9pY2UiOiAiQ2VudGVyIiwgIkNhcExlZnRDaG9pY2UiOiAiKCIsICJDYXBSaWdodENob2ljZSI6ICI+IiwgIkZvbnRDb21ib0JveCI6ICJtcGx1cy0xbW4tbWVkaXVtIiwgIkhlaWdodEN0cmwiOiAiMSIsICJMYXllckNvbWJvQm94IjogIkYuU2lsa1MiLCAiTXVsdGlMaW5lVGV4dCI6ICJDQU5SWF9XSUZJIiwgIlBhZGRpbmdCb3R0b21DdHJsIjogIiIsICJQYWRkaW5nTGVmdEN0cmwiOiAiIiwgIlBhZGRpbmdSaWdodEN0cmwiOiAiIiwgIlBhZGRpbmdUb3BDdHJsIjogIiIsICJXaWR0aEN0cmwiOiAiIn0=")
@@
 	(footprint "kibuzzard-6618272A"
 		(layer "F.Cu")
-		(at 124.6 86.73)
+		(at 124.25 81.625)
 		(descr "Generated with KiBuzzard")
 		(tags "kb_params=eyJBbGlnbm1lbnRDaG9pY2UiOiAiQ2VudGVyIiwgIkNhcExlZnRDaG9pY2UiOiAiKCIsICJDYXBSaWdodENob2ljZSI6ICI+IiwgIkZvbnRDb21ib0JveCI6ICJtcGx1cy0xbW4tbWVkaXVtIiwgIkhlaWdodEN0cmwiOiAiMSIsICJMYXllckNvbWJvQm94IjogIkYuU2lsa1MiLCAiTXVsdGlMaW5lVGV4dCI6ICJDQU5UWF9NSU5JTUEiLCAiUGFkZGluZ0JvdHRvbUN0cmwiOiAiIiwgIlBhZGRpbmdMZWZ0Q3RybCI6ICIiLCAiUGFkZGluZ1JpZ2h0Q3RybCI6ICIiLCAiUGFkZGluZ1RvcEN0cmwiOiAiIiwgIldpZHRoQ3RybCI6ICIifQ==")
@@
 	)
 	(segment
-		(start 132.315 79.08)
-		(end 130.05 79.08)
-		(width 0.3)
-		(layer "B.Cu")
-		(net 11)
-	)
-	(segment
-		(start 130.05 79.08)
-		(end 128.89 77.92)
-		(width 0.3)
-		(layer "B.Cu")
-		(net 11)
-	)
-	(segment
-		(start 128.89 77.92)
-		(end 128.89 49.266)
+		(start 132.315 84.08)
+		(end 128.956 80.721)
 		(width 0.3)
-		(layer "B.Cu")
+		(layer "F.Cu")
 		(net 11)
 	)
 	(segment
-		(start 128.89 49.266)
+		(start 128.956 80.721)
 		(end 128.956 49.2)
 		(width 0.3)
-		(layer "B.Cu")
+		(layer "F.Cu")
 		(net 11)
 	)
 	(segment
-		(start 127.21 58.09)
-		(end 129.12 56.18)
+		(start 132.315 79.08)
+		(end 132.315 53.461)
 		(width 0.3)
 		(layer "F.Cu")
@@
 	)
 	(segment
-		(start 136.6 49.224)
+		(start 132.315 53.461)
 		(end 136.576 49.2)
 		(width 0.3)
@@
 	)
 	(segment
-		(start 127.21 82.97)
-		(end 127.21 58.09)
-		(width 0.3)
-		(layer "F.Cu")
-		(net 17)
-	)
-	(segment
-		(start 136.6 55.1)
-		(end 136.6 49.224)
-		(width 0.3)
-		(layer "F.Cu")
-		(net 17)
-	)
-	(segment
-		(start 129.12 56.18)
-		(end 135.52 56.18)
-		(width 0.3)
-		(layer "F.Cu")
-		(net 17)
-	)
-	(segment
-		(start 132.315 84.08)
-		(end 128.32 84.08)
-		(width 0.3)
-		(layer "F.Cu")
-		(net 17)
-	)
-	(segment
-		(start 128.32 84.08)
-		(end 127.21 82.97)
-		(width 0.3)
-		(layer "F.Cu")
-		(net 17)
-	)
-	(segment
-		(start 135.52 56.18)
-		(end 136.6 55.1)
-		(width 0.3)
-		(layer "F.Cu")
-		(net 17)
-	)
-	(segment
-		(start 153.34 49.22)
-		(end 153.34 49.2)
-		(width 0.25)
-		(layer "F.Cu")
-		(net 19)
-	)
-	(segment
-		(start 132.315 88.425)
-		(end 133.45 89.56)
-		(width 0.3)
-		(layer "B.Cu")
-		(net 19)
-	)
-	(segment
-		(start 133.45 89.56)
-		(end 140.21 89.56)
-		(width 0.3)
-		(layer "B.Cu")
-		(net 19)
-	)
-	(segment
-		(start 142.9 56.12)
-		(end 151.76 56.12)
+		(start 132.315 81.58)
+		(end 133.515 80.38)
 		(width 0.3)
 		(layer "B.Cu")
@@
 	)
 	(segment
-		(start 140.21 89.56)
-		(end 141.38 88.39)
+		(start 150.005761 50.425)
+		(end 152.115 50.425)
 		(width 0.3)
 		(layer "B.Cu")
@@
 	)
 	(segment
-		(start 153.34 54.54)
+		(start 152.115 50.425)
 		(end 153.34 49.2)
 		(width 0.3)
@@
 	)
 	(segment
-		(start 141.38 88.39)
-		(end 141.38 57.64)
+		(start 133.515 66.915761)
+		(end 150.005761 50.425)
 		(width 0.3)
 		(layer "B.Cu")
@@
 	)
 	(segment
-		(start 132.315 86.58)
-		(end 132.315 88.425)
-		(width 0.3)
-		(layer "B.Cu")
-		(net 19)
-	)
-	(segment
-		(start 141.38 57.64)
-		(end 142.9 56.12)
-		(width 0.3)
-		(layer "B.Cu")
-		(net 19)
-	)
-	(segment
-		(start 151.76 56.12)
-		(end 153.34 54.54)
+		(start 133.515 80.38)
+		(end 133.515 66.915761)
 		(width 0.3)
 		(layer "B.Cu")
@@
 	)
 	(segment
-		(start 127.71 60.71)
-		(end 130.15 58.27)
+		(start 129.06 70.097057)
+		(end 149.957057 49.2)
 		(width 0.3)
-		(layer "F.Cu")
+		(layer "B.Cu")
 		(net 22)
 	)
 	(segment
-		(start 128.9 81.58)
-		(end 127.71 80.39)
+		(start 132.315 86.58)
+		(end 129.06 83.325)
 		(width 0.3)
-		(layer "F.Cu")
+		(layer "B.Cu")
 		(net 22)
 	)
 	(segment
-		(start 150.8 56.87)
+		(start 149.957057 49.2)
 		(end 150.8 49.2)
 		(width 0.3)
-		(layer "F.Cu")
-		(net 22)
-	)
-	(segment
-		(start 130.15 58.27)
-		(end 149.4 58.27)
-		(width 0.3)
-		(layer "F.Cu")
-		(net 22)
-	)
-	(segment
-		(start 149.4 58.27)
-		(end 150.8 56.87)
-		(width 0.3)
-		(layer "F.Cu")
-		(net 22)
-	)
-	(segment
-		(start 127.71 80.39)
-		(end 127.71 60.71)
-		(width 0.3)
-		(layer "F.Cu")
+		(layer "B.Cu")
 		(net 22)
 	)
 	(segment
-		(start 132.315 81.58)
-		(end 128.9 81.58)
+		(start 129.06 83.325)
+		(end 129.06 70.097057)
 		(width 0.3)
-		(layer "F.Cu")
+		(layer "B.Cu")
 		(net 22)
 	)
@@
 	)
 	(segment
-		(start 134.855 84.16)
-		(end 134.855 86.54)
-		(width 0.3)
-		(layer "F.Cu")
-		(net 29)
-	)
-	(segment
-		(start 135.5 84.805)
-		(end 134.855 84.16)
-		(width 0.3)
-		(layer "F.Cu")
-		(net 29)
-	)
-	(segment
-		(start 134.855 86.54)
-		(end 134.815 86.58)
-		(width 0.3)
-		(layer "F.Cu")
-		(net 29)
-	)
-	(segment
 		(start 144.375 84.805)
 		(end 135.5 84.805)
@@
 	)
 	(segment
-		(start 135.4 80.995)
-		(end 134.815 81.58)
-		(width 0.3)
-		(layer "F.Cu")
-		(net 34)
-	)
-	(segment
-		(start 134.815 79.08)
-		(end 134.815 81.58)
-		(width 0.3)
-		(layer "F.Cu")
-		(net 34)
-	)
-	(segment

Commit message: fix: change routing
Parts:
- moved kibuzzard-661826C2 0.23 mm to (139.7, 81.4)
- moved kibuzzard-661826AE 0.15 mm to (139.7, 84.2)
Routing:
- net +3V3: track 25.3 -> 0.00 mm, vias 1 -> 0
- net +5V: track 22.4 -> 28.2 mm
- net Net-(J5-Pin_5): track 8.88 -> 12.2 mm
- net Net-(J5-Pin_7): track 8.97 -> 12.3 mm
Changed lines of the file:
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@@
 	(footprint "kibuzzard-661826C2"
 		(layer "F.Cu")
-		(at 139.425 81.45)
+		(at 139.65 81.4)
 		(descr "Generated with KiBuzzard")
 		(tags "kb_params=eyJBbGlnbm1lbnRDaG9pY2UiOiAiQ2VudGVyIiwgIkNhcExlZnRDaG9pY2UiOiAiPCIsICJDYXBSaWdodENob2ljZSI6ICIpIiwgIkZvbnRDb21ib0JveCI6ICJtcGx1cy0xbW4tbWVkaXVtIiwgIkhlaWdodEN0cmwiOiAiMSIsICJMYXllckNvbWJvQm94IjogIkYuU2lsa1MiLCAiTXVsdGlMaW5lVGV4dCI6ICJDQU5UWCIsICJQYWRkaW5nQm90dG9tQ3RybCI6ICIiLCAiUGFkZGluZ0xlZnRDdHJsIjogIiIsICJQYWRkaW5nUmlnaHRDdHJsIjogIiIsICJQYWRkaW5nVG9wQ3RybCI6ICIiLCAiV2lkdGhDdHJsIjogIiJ9")
@@
 	(footprint "kibuzzard-661826AE"
 		(layer "F.Cu")
-		(at 139.55 84.25)
+		(at 139.7 84.225)
 		(descr "Generated with KiBuzzard")
 		(tags "kb_params=eyJBbGlnbm1lbnRDaG9pY2UiOiAiQ2VudGVyIiwgIkNhcExlZnRDaG9pY2UiOiAiPCIsICJDYXBSaWdodENob2ljZSI6ICIpIiwgIkZvbnRDb21ib0JveCI6ICJtcGx1cy0xbW4tbWVkaXVtIiwgIkhlaWdodEN0cmwiOiAiMSIsICJMYXllckNvbWJvQm94IjogIkYuU2lsa1MiLCAiTXVsdGlMaW5lVGV4dCI6ICJDQU5SWCIsICJQYWRkaW5nQm90dG9tQ3RybCI6ICIiLCAiUGFkZGluZ0xlZnRDdHJsIjogIiIsICJQYWRkaW5nUmlnaHRDdHJsIjogIiIsICJQYWRkaW5nVG9wQ3RybCI6ICIiLCAiV2lkdGhDdHJsIjogIiJ9")
@@
 	)
 	(segment
+		(start 149.325 84.805)
+		(end 149.325 87.5575)
+		(width 0.4)
+		(layer "F.Cu")
+		(net 3)
+	)
+	(segment
 		(start 146.2675 87.57)
 		(end 146.2675 91.7325)
@@
 	)
 	(segment
+		(start 149.32 87.5775)
+		(end 149.3125 87.57)
+		(width 0.4)
+		(layer "F.Cu")
+		(net 3)
+	)
+	(segment
+		(start 149.325 87.5575)
+		(end 149.3125 87.57)
+		(width 0.4)
+		(layer "F.Cu")
+		(net 3)
+	)
+	(segment
 		(start 146.2675 87.57)
 		(end 146.2675 84.2175)
@@
 	)
 	(segment
+		(start 149.3125 87.57)
+		(end 146.2675 87.57)
+		(width 0.4)
+		(layer "F.Cu")
+		(net 3)
+	)
+	(segment
 		(start 145.33 92.67)
 		(end 139.2 92.67)
@@
 	)
 	(segment
-		(start 132.315 81.58)
-		(end 133.515 80.38)
+		(start 150.005761 50.425)
+		(end 133.515 66.915761)
 		(width 0.3)
 		(layer "B.Cu")
@@
 	)
 	(segment
-		(start 150.005761 50.425)
-		(end 152.115 50.425)
+		(start 152.115 50.425)
+		(end 150.005761 50.425)
 		(width 0.3)
 		(layer "B.Cu")
@@
 	)
 	(segment
-		(start 152.115 50.425)
-		(end 153.34 49.2)
+		(start 133.515 80.38)
+		(end 132.315 81.58)
 		(width 0.3)
 		(layer "B.Cu")
@@
 	)
 	(segment
-		(start 133.515 66.915761)
-		(end 150.005761 50.425)
+		(start 153.34 49.2)
+		(end 152.115 50.425)
 		(width 0.3)
 		(layer "B.Cu")
@@
 	)
 	(segment
-		(start 133.515 80.38)
-		(end 133.515 66.915761)
+		(start 133.515 66.915761)
+		(end 133.515 80.38)
 		(width 0.3)
 		(layer "B.Cu")
@@
 	)
 	(segment
-		(start 129.06 70.097057)
-		(end 149.957057 49.2)
+		(start 150.523654 49.2)
+		(end 129.06 70.663655)
 		(width 0.3)
 		(layer "B.Cu")
@@
 	)
 	(segment
-		(start 132.315 86.58)
-		(end 129.06 83.325)
+		(start 150.8 49.2)
+		(end 150.523654 49.2)
 		(width 0.3)
 		(layer "B.Cu")
@@
 	)
 	(segment
-		(start 149.957057 49.2)
-		(end 150.8 49.2)
+		(start 129.06 83.325)
+		(end 129.06 70.663655)
 		(width 0.3)
 		(layer "B.Cu")
@@
 	)
 	(segment
-		(start 129.06 83.325)
-		(end 129.06 70.097057)
+		(start 132.315 86.58)
+		(end 129.06 83.325)
 		(width 0.3)
 		(layer "B.Cu")
@@
 	)
 	(segment
-		(start 149.325 84.805)
-		(end 149.325 87.5575)
-		(width 0.4)
-		(layer "F.Cu")
-		(net 26)
-	)
-	(segment
-		(start 149.32 93.01)
-		(end 149.32 87.5775)
-		(width 0.4)
-		(layer "F.Cu")
-		(net 26)
-	)
-	(segment
-		(start 148.36 93.97)
-		(end 149.32 93.01)
-		(width 0.4)
+		(start 134.855 84.16)
+		(end 134.855 86.54)
+		(width 0.3)
 		(layer "F.Cu")
-		(net 26)
+		(net 29)
 	)
 	(segment
-		(start 145.6 93.97)
-		(end 148.36 93.97)
-		(width 0.4)
+		(start 143.92 84.35)
+		(end 135.045 84.35)
+		(width 0.3)
 		(layer "F.Cu")
-		(net 26)
+		(net 29)
 	)
 	(segment
-		(start 149.32 87.5775)
-		(end 149.3125 87.57)
-		(width 0.4)
+		(start 135.045 84.35)
+		(end 134.855 84.16)
+		(width 0.3)
 		(layer "F.Cu")
-		(net 26)
+		(net 29)
 	)
 	(segment
-		(start 149.325 87.5575)
-		(end 149.3125 87.57)
-		(width 0.4)
+		(start 134.855 86.54)
+		(end 134.815 86.58)
+		(width 0.3)
 		(layer "F.Cu")
-		(net 26)
-	)
-	(via
-		(at 145.6 93.97)
-		(size 0.6)
-		(drill 0.3)
-		(layers "F.Cu" "B.Cu")
-		(net 26)
-	)
-	(segment
-		(start 145.6 93.97)
-		(end 136.49 93.97)
-		(width 0.4)
-		(layer "B.Cu")
-		(net 26)
-	)
-	(segment
-		(start 136.49 93.97)
-		(end 135.56 94.9)
-		(width 0.4)
-		(layer "B.Cu")
-		(net 26)
-	)
-	(segment
-		(start 135.56 94.9)
-		(end 135.56 97.46)
-		(width 0.4)
-		(layer "B.Cu")
-		(net 26)
+		(net 29)
 	)
 	(segment
 		(start 144.375 84.805)
-		(end 135.5 84.805)
+		(end 143.92 84.35)
 		(width 0.3)
 		(layer "F.Cu")
@@
 	)
 	(segment
+		(start 134.815 81.58)
+		(end 134.815 79.08)
+		(width 0.3)
+		(layer "F.Cu")
+		(net 34)
+	)
+	(segment
+		(start 143.97 81.4)
+		(end 134.995 81.4)
+		(width 0.3)
+		(layer "F.Cu")
+		(net 34)
+	)
+	(segment
 		(start 144.375 80.995)
-		(end 135.4 80.995)
+		(end 143.97 81.4)
+		(width 0.3)
+		(layer "F.Cu")
+		(net 34)
+	)
+	(segment
+		(start 134.995 81.4)
+		(end 134.815 81.58)
 		(width 0.3)
 		(layer "F.Cu")
