File: CANBus/Hardware/CAN_Shield_UNO/CAN_Shield_UNO.kicad_pcb (KiCad board)
At the start: 2 copper layers, 68.6 x 53.3 mm, 39 parts, among them J1 Power, J2 Digital/PWM, J3 Analog, J4 Digital/PWM, J7 Screw_Terminal_01x02, U2 TCAN1051HGV

Commit message: fix: change labels (v1.1)
Parts:
- removed kibuzzard-6618216B (x2): G***, kibuzzard-6618216B
- added kibuzzard-667B328E: G***, kibuzzard-667B328E, B.Cu at (134.0, 74.4)
- added kibuzzard-667B3298: G***, kibuzzard-667B3298, F.Cu at (133.5, 74.0)
